File: hardware/crawler_schematic/crawler_schematic.kicad_sch (KiCad schematic)
At the start: 11 parts, among them J1 Conn_01x02_Pin, J2 MP1584 Buck Converter, M1 Motor_DC, M2 Motor_Servo, U1 NRF24L01

Commit message: update: update kicad schem for h bridge power
Connections:
- net at TB6612_HBridge.GND (Pin_15): now also STM32F411_BlackPill.G (Pin_39)
- net at STM32F411_BlackPill.G (Pin_39): now also C1.2, C2.2, J2.OUT- (Pin_2), R1.2, U1.1 (GND); no longer TB6612_HBridge.GND (Pin_15)
Changed lines of the file:
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@@
-	)
-	(junction
-		(at 182.88 81.28)
-		(diameter 0)
-		(color 0 0 0 0)
 	)
 	(junction
@@
 	)
 	(junction
+		(at 149.86 76.2)
+		(diameter 0)
+		(color 0 0 0 0)
+	)
+	(junction
 		(at 121.92 74.93)
 		(diameter 0)
@@
 	)
 	(junction
+		(at 152.4 78.74)
+		(diameter 0)
+		(color 0 0 0 0)
+	)
+	(junction
 		(at 142.24 36.83)
 		(diameter 0)
@@
 	(wire
 		(pts
-			(xy 161.29 76.2) (xy 148.59 76.2)
+			(xy 161.29 76.2) (xy 149.86 76.2)
 		)
 		(stroke
@@
 	(wire
 		(pts
-			(xy 58.42 116.84) (xy 182.88 116.84)
-		)
-		(stroke
-			(width 0)
-			(type default)
-		)
-	)
-	(wire
-		(pts
 			(xy 50.8 95.25) (xy 50.8 77.47)
 		)
@@
 	(wire
 		(pts
+			(xy 149.86 111.76) (xy 149.86 76.2)
+		)
+		(stroke
+			(width 0)
+			(type default)
+		)
+	)
+	(wire
+		(pts
 			(xy 165.1 67.31) (xy 142.24 67.31)
 		)
@@
 	(wire
 		(pts
+			(xy 149.86 76.2) (xy 148.59 76.2)
+		)
+		(stroke
+			(width 0)
+			(type default)
+		)
+	)
+	(wire
+		(pts
 			(xy 73.66 80.01) (xy 78.74 80.01)
 		)
@@
 	(wire
 		(pts
-			(xy 182.88 81.28) (xy 182.88 116.84)
+			(xy 60.96 111.76) (xy 149.86 111.76)
 		)
 		(stroke
@@
 	(wire
 		(pts
+			(xy 58.42 116.84) (xy 152.4 116.84)
+		)
+		(stroke
+			(width 0)
+			(type default)
+		)
+	)
+	(wire
+		(pts
 			(xy 173.99 81.28) (xy 161.29 81.28)
 		)
@@
 	(wire
 		(pts
-			(xy 191.77 71.12) (xy 173.99 71.12)
-		)
-		(stroke
-			(width 0)
-			(type default)
-		)
-	)
-	(wire
-		(pts
 			(xy 67.31 64.77) (xy 78.74 64.77)
 		)
@@
 	(wire
 		(pts
-			(xy 191.77 111.76) (xy 191.77 71.12)
-		)
-		(stroke
-			(width 0)
-			(type default)
-		)
-	)
-	(wire
-		(pts
 			(xy 48.26 90.17) (xy 53.34 90.17)
 		)
@@
 	(wire
 		(pts
+			(xy 152.4 116.84) (xy 152.4 78.74)
+		)
+		(stroke
+			(width 0)
+			(type default)
+		)
+	)
+	(wire
+		(pts
 			(xy 48.26 100.33) (xy 26.67 100.33)
 		)
@@
 	(wire
 		(pts
-			(xy 161.29 78.74) (xy 148.59 78.74)
+			(xy 152.4 78.74) (xy 148.59 78.74)
+		)
+		(stroke
+			(width 0)
+			(type default)
+		)
+	)
+	(wire
+		(pts
+			(xy 161.29 78.74) (xy 152.4 78.74)
 		)
 		(stroke
@@
 		)
 		(stroke
-			(width 0)
-			(type default)
-		)
-	)
-	(wire
-		(pts
-			(xy 60.96 111.76) (xy 191.77 111.76)
-		)
-		(stroke

Commit message: update: update crawler schematic for servo pwm to pb4
Connections:
- net at TB6612_HBridge.GND (Pin_15): now also STM32F411_BlackPill.G (Pin_39)
- net at STM32F411_BlackPill.G (Pin_39): now also C1.2, C2.2, J2.OUT- (Pin_2), R1.2, U1.1 (GND); no longer TB6612_HBridge.GND (Pin_15)
- net at M2.1 (PWM): now also STM32F411_BlackPill.B4 (Pin_12); no longer STM32F411_BlackPill.B12
- net at 2S_Lipo.1 (+), J1.VMot+ (Pin_1), J2.IN+ (Pin_4): no longer M2.2 (+)
- net at 2S_Lipo.2 (-), J1.VMoT- (Pin_2), J2.IN- (Pin_3): no longer M2.3 (-)
- net at J2.OUT+ (Pin_1), R1.1, STM32F411_BlackPill.5V (Pin_40): now also M2.2 (+), M2.3 (-)
Changed lines of the file:
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@@
+	)
+	(junction
+		(at 115.57 31.75)
+		(diameter 0)
+		(color 0 0 0 0)
 	)
 	(junction
@@
 	)
 	(junction
-		(at 173.99 81.28)
-		(diameter 0)
-		(color 0 0 0 0)
-	)
-	(junction
-		(at 173.99 71.12)
+		(at 109.22 31.75)
 		(diameter 0)
 		(color 0 0 0 0)
@@
 	(wire
 		(pts
+			(xy 115.57 24.13) (xy 115.57 31.75)
+		)
+		(stroke
+			(width 0)
+			(type default)
+		)
+	)
+	(wire
+		(pts
+			(xy 66.04 85.09) (xy 67.31 85.09)
+		)
+		(stroke
+			(width 0)
+			(type default)
+		)
+	)
+	(wire
+		(pts
+			(xy 69.85 69.85) (xy 78.74 69.85)
+		)
+		(stroke
+			(width 0)
+			(type default)
+		)
+	)
+	(wire
+		(pts
+			(xy 161.29 76.2) (xy 149.86 76.2)
+		)
+		(stroke
+			(width 0)
+			(type default)
+		)
+	)
+	(wire
+		(pts
+			(xy 109.22 67.31) (xy 142.24 67.31)
+		)
+		(stroke
+			(width 0)
+			(type default)
+		)
+	)
+	(wire
+		(pts
+			(xy 71.12 77.47) (xy 78.74 77.47)
+		)
+		(stroke
+			(width 0)
+			(type default)
+		)
+	)
+	(wire
+		(pts
+			(xy 161.29 81.28) (xy 161.29 78.74)
+		)
+		(stroke
+			(width 0)
+			(type default)
+		)
+	)
+	(wire
+		(pts
+			(xy 109.22 80.01) (xy 121.92 80.01)
+		)
+		(stroke
+			(width 0)
+			(type default)
+		)
+	)
+	(wire
+		(pts
+			(xy 91.44 34.29) (xy 109.22 34.29)
+		)
+		(stroke
+			(width 0)
+			(type default)
+		)
+	)
+	(wire
+		(pts
+			(xy 71.12 59.69) (xy 78.74 59.69)
+		)
+		(stroke
+			(width 0)
+			(type default)
+		)
+	)
+	(wire
+		(pts
+			(xy 48.26 92.71) (xy 48.26 100.33)
+		)
+		(stroke
+			(width 0)
+			(type default)
+		)
+	)
+	(wire
+		(pts
+			(xy 45.72 34.29) (xy 45.72 29.21)
+		)
+		(stroke
+			(width 0)
+			(type default)
+		)
+	)
+	(wire
+		(pts
+			(xy 34.29 20.32) (xy 109.22 20.32)
+		)
+		(stroke
+			(width 0)
+			(type default)
+		)
+	)
+	(wire
+		(pts
 			(xy 115.57 31.75) (xy 115.57 74.93)
 		)
@@
 	(wire
 		(pts
-			(xy 182.88 20.32) (xy 182.88 81.28)
-		)
-		(stroke
-			(width 0)
-			(type default)
-		)
-	)
-	(wire
-		(pts
-			(xy 66.04 85.09) (xy 67.31 85.09)
-		)
-		(stroke
-			(width 0)
-			(type default)
-		)
-	)
-	(wire
-		(pts
-			(xy 72.39 31.75) (xy 78.74 31.75)
-		)
-		(stroke
-			(width 0)
-			(type default)
-		)
-	)
-	(wire
-		(pts
-			(xy 69.85 69.85) (xy 78.74 69.85)
-		)
-		(stroke
-			(width 0)
-			(type default)
-		)
-	)
-	(wire
-		(pts
-			(xy 161.29 76.2) (xy 149.86 76.2)
-		)
-		(stroke
-			(width 0)
-			(type default)
-		)
-	)
-	(wire
-		(pts
-			(xy 109.22 67.31) (xy 142.24 67.31)
-		)
-		(stroke
-			(width 0)
-			(type default)
-		)
-	)
-	(wire
-		(pts
-			(xy 71.12 77.47) (xy 78.74 77.47)
-		)
-		(stroke
-			(width 0)
-			(type default)
-		)
-	)
-	(wire
-		(pts
-			(xy 161.29 81.28) (xy 161.29 78.74)
-		)
-		(stroke
-			(width 0)
-			(type default)
-		)
-	)
-	(wire
-		(pts
-			(xy 109.22 80.01) (xy 121.92 80.01)
-		)
-		(stroke
-			(width 0)
-			(type default)
-		)
-	)
-	(wire
-		(pts
-			(xy 91.44 34.29) (xy 109.22 34.29)
-		)
-		(stroke
-			(width 0)
-			(type default)
-		)
-	)
-	(wire
-		(pts
-			(xy 48.26 92.71) (xy 48.26 100.33)
-		)
-		(stroke
-			(width 0)
-			(type default)
-		)
-	)
-	(wire
-		(pts
 			(xy 50.8 95.25) (xy 50.8 77.47)
 		)
@@
 	(wire
 		(pts
-			(xy 173.99 24.13) (xy 173.99 71.12)
-		)
-		(stroke
-			(width 0)
-			(type default)
-		)
-	)
-	(wire
-		(pts
 			(xy 91.44 52.07) (xy 124.46 52.07)
 		)
@@
 	(wire
 		(pts
-			(xy 45.72 34.29) (xy 45.72 25.4)
-		)
-		(stroke
-			(width 0)
-			(type default)
-		)
-	)
-	(wire
-		(pts
 			(xy 48.26 87.63) (xy 48.26 90.17)
 		)
@@
 	(wire
 		(pts
+			(xy 109.22 31.75) (xy 115.57 31.75)
+		)
+		(stroke
+			(width 0)
+			(type default)
+		)
+	)
+	(wire
+		(pts
 			(xy 50.8 77.47) (xy 71.12 77.47)
 		)
@@
 	(wire
 		(pts
+			(xy 71.12 29.21) (xy 71.12 59.69)
+		)
+		(stroke
+			(width 0)
+			(type default)
+		)
+	)
+	(wire
+		(pts
 			(xy 26.67 87.63) (xy 48.26 87.63)
 		)
@@
 	(wire
 		(pts
-			(xy 182.88 81.28) (xy 173.99 81.28)
-		)
-		(stroke
-			(width 0)
-			(type default)
-		)
-	)
-	(wire
-		(pts
 			(xy 153.67 50.8) (xy 165.1 50.8)
 		)
@@
 	(wire
 		(pts
-			(xy 91.44 31.75) (xy 115.57 31.75)
+			(xy 91.44 31.75) (xy 109.22 31.75)
 		)
 		(stroke
@@
 	(wire
 		(pts
-			(xy 34.29 20.32) (xy 182.88 20.32)
+			(xy 45.72 29.21) (xy 71.12 29.21)
 		)
 		(stroke
@@
 	(wire
 		(pts
+			(xy 38.1 24.13) (xy 115.57 24.13)
+		)
+		(stroke
+			(width 0)
+			(type default)
+		)
+	)
+	(wire
+		(pts
 			(xy 48.26 90.17) (xy 53.34 90.17)
 		)
@@
 	(wire
 		(pts
+			(xy 109.22 20.32) (xy 109.22 31.75)
+		)
+		(stroke
+			(width 0)
+			(type default)
+		)
+	)
+	(wire
+		(pts
 			(xy 161.29 78.74) (xy 152.4 78.74)
 		)
@@
 	(wire
 		(pts
-			(xy 72.39 25.4) (xy 72.39 31.75)
-		)
-		(stroke
-			(width 0)
-			(type default)
-		)
-	)
-	(wire
-		(pts
 			(xy 153.67 44.45) (xy 153.67 43.18)
 		)
@@
 	(wire
 		(pts
-			(xy 38.1 24.13) (xy 173.99 24.13)
-		)
-		(stroke
-			(width 0)
-			(type default)
-		)
-	)
-	(wire
-		(pts
 			(xy 121.92 74.93) (xy 133.35 74.93)
 		)
@@
 		)
 		(stroke
-			(width 0)
-			(type default)
-		)
-	)
-	(wire
-		(pts
-			(xy 45.72 25.4) (xy 72.39 25.4)
-		)
-		(stroke

Commit message: update: schematic cleanups
Parts:
- added SW?: switch, Button_Switch_SMD:Nidec_Copal_CAS-120A, symbol Switch:SW_Nidec_CAS-120A1
Connections:
- net at TB6612_HBridge.GND (Pin_15): now also STM32F411_BlackPill.G (Pin_39)
- net at STM32F411_BlackPill.G (Pin_39): now also C1.2, C2.2, J2.OUT+ (Pin_1), M2.3 (-), R1.2, U1.1 (GND); no longer TB6612_HBridge.GND (Pin_15)
- net at TB6612_HBridge.STBY (Pin_7), TB6612_HBridge.VCC (Pin_2): now also STM32F411_BlackPill.5V (Pin_40); no longer STM32F411_BlackPill.3V3 (Pin_38)
- net at M2.2 (+), R1.1, STM32F411_BlackPill.5V (Pin_40): now also J2.OUT- (Pin_2); no longer J2.OUT+ (Pin_1), M2.3 (-)
- net at J1.VMot+ (Pin_1), J2.IN+ (Pin_4): now also SW?.3 (A); no longer 2S_Lipo.1 (+)
- new net: 2S_Lipo.1 (+), SW?.2 (B)
Other:
- note added: "NOTE: jump stby to vcc+"
- moved on the sheet: 2S_Lipo
