File: hardware/crawler_schematic/crawler_schematic.kicad_sch (KiCad schematic)
At the start: 32 parts, among them J1 JST-PH, J3 SWD_Header, M2 Motor_Servo, U1 STM32F411CEUx, U2 RY8336, U2 TB6612FNG, U3 RY8336

Commit message: update: MITE completion 80%
Parts:
- removed C?: 104nF, Capacitor_SMD:C_1206_3216Metric, symbol Device:C_Small
- removed C?: 10uF, Capacitor_SMD:C_1206_3216Metric, symbol Device:C_Polarized
- removed U?: NRF24L01, RF_Module:nRF24L01_Breakout, symbol RF:NRF24L01_Breakout
- added AE1: 50ohm, RF_Antenna:Johanson_2450AT43F0100, symbol Device:Antenna
- added C_H_3: 47uF, Capacitor_SMD:CP_Elec_6.3x5.4, symbol Device:C_Polarized
- added C_M_1, C_M_2: 4.3pF, Capacitor_SMD:C_0603_1608Metric, symbol Device:C_Small
- added C_M_3: 2.2uF, Capacitor_SMD:C_0603_1608Metric, symbol Device:C_Small
- added C_M_4, C_M_5, C_M_6: 100 nF, X7R, 16 V, C_0402_1005Metric, symbol Device:C_Small
- added C_M_7: 100 nF, X7R, Capacitor_SMD:C_0402_1005Metric, symbol Device:C_Small
- added C_nrf_1, C_nrf_11: 10nF, Capacitor_SMD:C_0402_1005Metric, symbol Device:C_Small
- added C_nrf_2: 1nF, Capacitor_SMD:C_0402_1005Metric, symbol Device:C_Small
- added C_nrf_3: 33nF, Capacitor_SMD:C_0402_1005Metric, symbol Device:C_Small
- added C_nrf_4: 1.0pF, Capacitor_SMD:C_0402_1005Metric, symbol Device:C_Small
- added C_nrf_5: 1.5pF, Capacitor_SMD:C_0402_1005Metric, symbol Device:C_Small
- added C_nrf_6: 4.7pF, Capacitor_SMD:C_0402_1005Metric, symbol Device:C_Small
- added C_nrf_7: 2.2nF, Capacitor_SMD:C_0402_1005Metric, symbol Device:C_Small
- added C_nrf_8, C_nrf_9: 22pF, Capacitor_SMD:C_0402_1005Metric, symbol Device:C_Small
- added C_ref_1, C_ref_2, C_ref_3, C_ref_4: Opt., Capacitor_SMD:C_0603_1608Metric, symbol Device:C_Small
- added C_rst_1: 100nF, Capacitor_SMD:C_0603_1608Metric, symbol Device:C_Small
- added D_L_1: LED_pc13, LED_SMD:LED_0805_2012Metric, symbol Device:LED_Small
- added D_L_2: LED_pwr, LED_SMD:LED_0805_2012Metric, symbol Device:LED_Small
- added L_M_1: 10uH +-10%, Inductor_SMD:L_0603_1608Metric, symbol Device:L
- added L_nrf_1: 8.2nH, Inductor_SMD:L_0402_1005Metric, symbol Device:L
- added L_nrf_2: 3.9nH, Inductor_SMD:L_0402_1005Metric, symbol Device:L
- added L_nrf_3: 2.7nH, Inductor_SMD:L_0402_1005Metric, symbol Device:L
- added R_B_1, R_B_2: 10K, Resistor_SMD:R_0603_1608Metric, symbol Device:R_Small_US
- added R_L_1: 1K, Resistor_SMD:R_0603_1608Metric, symbol Device:R_Small_US
- added R_L_2: 5.1K, Resistor_SMD:R_0603_1608Metric, symbol Device:R_Small_US
- added R_nrf_1: 22k, Resistor_SMD:R_0201_0603Metric, symbol Device:R_Small_US
- added R_nrf_2: 1M, Resistor_SMD:R_0201_0603Metric, symbol Device:R_Small_US
- added R_rst_1: NC, Resistor_SMD:R_0603_1608Metric, symbol Device:R_Small_US
- added SW_B_1: boot switch, Button_Switch_SMD:SW_Push_1P1T_NO_CK_KMR2, symbol Switch:SW_SPST
- added SW_rst_2: nrst_switch, Button_Switch_SMD:SW_Push_1P1T_NO_CK_KMR2, symbol Switch:SW_SPST
- added U6: NRF24L01, Package_DFN_QFN:QFN-20-1EP_4x5mm_P0.5mm_EP2.65x3.65mm_ThermalVias, symbol RF:NRF24L01
- added Y_M_1, Y_nrf_1: Crystal_4pin_GND24, Crystal:Crystal_SMD_3225-4Pin_3.2x2.5mm, symbol my_symbols:Crystal_4pin_GND24
- C1_3.3: renamed from C1_3.?; footprint Capacitor_SMD:C_1206_3216Metric -> Capacitor_SMD:C_0603_1608Metric
- C1_5: renamed from C1_?; footprint Capacitor_SMD:C_1206_3216Metric -> Capacitor_SMD:C_0603_1608Metric
- CFF_3.3: renamed from CFF_3.?; footprint Capacitor_SMD:C_1206_3216Metric -> Capacitor_SMD:C_0603_1608Metric
- CFF_5: renamed from CFF_?; footprint Capacitor_SMD:C_1206_3216Metric -> Capacitor_SMD:C_0603_1608Metric
- CIN_3.3: renamed from CIN_3.?; footprint Capacitor_SMD:C_1206_3216Metric -> Capacitor_SMD:C_0603_1608Metric
- CIN_5: renamed from CIN_?; footprint Capacitor_SMD:C_1206_3216Metric -> Capacitor_SMD:C_0603_1608Metric
- COUT_3.3: renamed from COUT_3.?; footprint Capacitor_SMD:C_1206_3216Metric -> Capacitor_SMD:C_0603_1608Metric
- COUT_5: renamed from COUT_?; footprint Capacitor_SMD:C_1206_3216Metric -> Capacitor_SMD:C_0603_1608Metric
- C_H_1, C_H_2: renamed from C?; footprint Capacitor_SMD:C_1206_3216Metric -> Capacitor_SMD:C_0603_1608Metric
- J3: footprint Package_DFN_QFN:WDFN-10-1EP_3x3mm_P0.5mm_EP1.8x2.5mm -> Connector_PinHeader_2.54mm:PinHeader_1x04_P2.54mm_Vertical
- L1_3.3: renamed from L1_3.?; footprint Inductor_SMD:L_Cenker_CKCS8040 -> easyeda2kicad:IND-SMD_L3.0-W3.0_FTC303020D
- L1_5: renamed from L1_?; footprint Inductor_SMD:L_Cenker_CKCS8040 -> easyeda2kicad:IND-SMD_L3.0-W3.0_FTC303020D
- R1_3.3: renamed from R1_3.?; footprint Resistor_SMD:R_0201_0603Metric -> Resistor_SMD:R_0603_1608Metric
- R1_5, R_H_1: renamed from R?; footprint Resistor_SMD:R_0201_0603Metric -> Resistor_SMD:R_0603_1608Metric
- R2_3.3: renamed from R2_3.?; footprint Resistor_SMD:R_0201_0603Metric -> Resistor_SMD:R_0603_1608Metric
- R2_5: renamed from R1_?; footprint Resistor_SMD:R_0201_0603Metric -> Resistor_SMD:R_0603_1608Metric
- R3_5: renamed from R2_?; footprint Resistor_SMD:R_0201_0603Metric -> Resistor_SMD:R_0603_1608Metric
- R_EN_3.3: renamed from R_EN_3.?; footprint Resistor_SMD:R_0201_0603Metric -> Resistor_SMD:R_0603_1608Metric
- R_EN_5: renamed from R_EN_?; footprint Resistor_SMD:R_0201_0603Metric -> Resistor_SMD:R_0603_1608Metric
- gave numbers to parts that had none: 1
- renumbered J1 to J2, U2 to U4
Connections:
- net IRQ is gone; now on net MISO: U1.13 (PA3)
- net +3.3V: now also U1.1 (VBAT), U1.24 (VDD), U1.36 (VDD), U1.48 (VDD), C_M_4.2, C_M_5.2, C_M_6.2, C_M_7.2, C_nrf_1.1, C_nrf_11.1, C_nrf_2.1, C_ref_1.1, C_ref_2.1, C_ref_3.1, L_M_1.2, R_L_1.2, R_L_2.2, R_rst_1.1, SW_B_1.2 (B), U6.15 (VDD), U6.18 (VDD), U6.7 (VDD)
- net +5V: now also M2.2 (+)
- net +BATT: now also C_H_3.1
- net AIN1: now also U1.42 (PB6); no longer U1.43 (PB7)
- net AIN2: now also U1.41 (PB5); no longer U1.45 (PB8)
- net GND: now also M2.3 (-), U1.23 (VSS), U1.35 (VSS), U1.47 (VSS), U1.49 (VSS), U1.8 (VSSA), C_H_3.2, C_M_1.1, C_M_2.1, C_M_3.1, C_M_4.1, C_M_5.1, C_M_6.1, C_M_7.1, C_nrf_1.2, C_nrf_11.2, C_nrf_2.2, C_nrf_3.2, C_nrf_4.2, C_nrf_6.1, C_nrf_7.1, C_nrf_8.2, C_nrf_9.2, C_ref_1.2, C_ref_2.2, C_ref_3.2, C_ref_4.2, C_rst_1.2, D_L_2.1 (K), R_B_1.2, R_B_2.1, R_nrf_1.2, SW_rst_2.2 (B), U6.14 (VSS), U6.17 (VSS), U6.20 (VSS), U6.8 (VSS), Y_M_1.2 (GND), Y_M_1.4 (GND), Y_nrf_1.2 (GND), Y_nrf_1.4 (GND)
- net MISO: now also U6.5 (MISO); no longer U1.16 (PA6)
- net MOSI: now also U1.14 (PA4), U6.4 (MOSI); no longer U1.17 (PA7)
- net PWMA: now also U1.40 (PB4); no longer U1.42 (PB6)
- net SCK: now also U6.3 (SCK)
- net servo_pwm: now also U1.43 (PB7); no longer U1.40 (PB4)
- net ~{CSN}: now also U1.16 (PA6), U6.2 (CSN); no longer U1.14 (PA4)
- net PC13: now reaches U1.2 (PC13)
- net PC13: now also D_L_1.1 (K)
- net PB2: now reaches U1.20 (PB2)
- net PB2: now also R_B_2.2
- net at U1.22 (VCAP1): now also C_M_3.2
- net BOOT0: now reaches U1.44 (BOOT0)
- net BOOT0: now also R_B_1.1, SW_B_1.1 (A)
- net at U1.5 (PH0): now also C_M_1.2, Y_M_1.1
- net at U1.6 (PH1): now also C_M_2.2, Y_M_1.3
- net NRST: now reaches U1.7 (NRST)
- net NRST: now also C_rst_1.1, R_rst_1.2, SW_rst_2.1 (A)
- net VREF+: now reaches U1.9 (VDDA)
- net VREF+: now also C_ref_4.1, L_M_1.1
- net BAT_IN: now reaches J1.1 (Pin_1), Q1.5 (D), Q1.6 (D), Q1.7 (D), Q1.8 (D)
- new net: AE1.1 (A), C_nrf_4.1, C_nrf_5.2
- new net: C_nrf_8.1, R_nrf_2.2, U6.9 (XC2), Y_nrf_1.1
- new net: D_L_2.2 (A), R_L_2.1
- new net: C_nrf_9.1, R_nrf_2.1, U6.10 (XC1), Y_nrf_1.3
- new net: D_L_1.2 (A), R_L_1.1
- new net: C_nrf_6.2, C_nrf_7.2, L_nrf_3.1, U6.11 (VDD_PA)
- new net: L_nrf_1.1, L_nrf_3.2, U6.12 (ANT1)
- new net: C_nrf_5.1, L_nrf_2.2
- new net: L_nrf_1.2, L_nrf_2.1, U6.13 (ANT2)
- new net: R_nrf_1.1, U6.16 (IREF)
- new net: C_nrf_3.1, U6.19 (DVDD)
- new net CE: U1.17 (PA7), U6.1 (CE)
- no-connect marks 10 -> 31
Other:
- removed sheet Power Sheet
- removed sheet stm32f411ce
- note added: "BOOT0"
- note added: "BUCK/POLARITY"
- note added: "H BRIDGE"
- note added: "JST/SERV0 OUT"
- note added: "LED"
- note added: "NRF24"
- note added: "NRF24L01 RF"
- note added: "NRST"
- note added: "SWD"
- title: (none) -> MITE v1
- moved on the sheet: J2, J3, M2, U1

Commit message: update: MITE v1 completion 80%
Changed lines of the file:
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@@
 		)
 		(property "Value" "NC"
-			(at 365.76 62.23 0)
+			(at 364.49 62.23 0)
 			(show_name no)
 			(do_not_autoplace no)
