File: hardware/crawler_schematic/power.kicad_sch (KiCad schematic)
At the start: 21 parts, among them J2 JST-PH, Q1 AO4407A, U5 RY8336

Commit message: update: schematic complete, start pcb design
Parts:
- C1_3.3, C1_5, CFF_3.3, CFF_5: footprint (none) -> Capacitor_SMD:C_1206_3216Metric
- R1_3.3, R1_5, R2_3.3, R2_5, R3, R_EN_3.3, R_EN_5: footprint Package_DIP:DIP-8_W7.62mm -> Resistor_SMD:R_0201_0603Metric
Changed lines of the file:
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@@
 			)
 		)
-		(property "Footprint" "Package_DIP:DIP-8_W7.62mm"
+		(property "Footprint" "Resistor_SMD:R_0201_0603Metric"
 			(at 153.67 77.47 0)
 			(hide yes)
@@
 			)
 		)
-		(property "Footprint" "Package_DIP:DIP-8_W7.62mm"
+		(property "Footprint" "Resistor_SMD:R_0201_0603Metric"
 			(at 105.41 114.3 0)
 			(hide yes)
@@
 			)
 		)
-		(property "Footprint" ""
+		(property "Footprint" "Capacitor_SMD:C_1206_3216Metric"
 			(at 132.08 66.04 0)
 			(hide yes)
@@
 			)
 		)
-		(property "Footprint" "Package_DIP:DIP-8_W7.62mm"
+		(property "Footprint" "Resistor_SMD:R_0201_0603Metric"
 			(at 154.94 120.65 0)
 			(hide yes)
@@
 			)
 		)
-		(property "Footprint" "Package_DIP:DIP-8_W7.62mm"
+		(property "Footprint" "Resistor_SMD:R_0201_0603Metric"
 			(at 154.94 132.08 0)
 			(hide yes)
@@
 			)
 		)
-		(property "Footprint" ""
+		(property "Footprint" "Capacitor_SMD:C_1206_3216Metric"
 			(at 163.83 121.92 0)
 			(hide yes)
@@
 			)
 		)
-		(property "Footprint" ""
+		(property "Footprint" "Capacitor_SMD:C_1206_3216Metric"
 			(at 133.35 109.22 0)
 			(hide yes)
@@
 			)
 		)
-		(property "Footprint" "Package_DIP:DIP-8_W7.62mm"
+		(property "Footprint" "Resistor_SMD:R_0201_0603Metric"
 			(at 57.15 88.9 0)
 			(hide yes)
@@
 			)
 		)
-		(property "Footprint" "Package_DIP:DIP-8_W7.62mm"
+		(property "Footprint" "Resistor_SMD:R_0201_0603Metric"
 			(at 104.14 71.12 0)
 			(hide yes)
@@
 			)
 		)
-		(property "Footprint" ""
+		(property "Footprint" "Capacitor_SMD:C_1206_3216Metric"
 			(at 162.56 78.74 0)
 			(hide yes)
@@
 			)
 		)
-		(property "Footprint" "Package_DIP:DIP-8_W7.62mm"
+		(property "Footprint" "Resistor_SMD:R_0201_0603Metric"
 			(at 153.67 88.9 0)
 			(hide yes)

Commit message: update: pcb work
Parts:
- L1_3.3, L1_5: footprint Package_SO:SOIC-20W_7.5x12.8mm_P1.27mm -> Inductor_SMD:L_Cenker_CKCS8040
Changed lines of the file:
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@@
 			)
 		)
-		(property "Footprint" "Package_SO:SOIC-20W_7.5x12.8mm_P1.27mm"
+		(property "Footprint" "Inductor_SMD:L_Cenker_CKCS8040"
 			(at 147.32 115.57 0)
 			(hide yes)
@@
 			)
 		)
-		(property "Footprint" "Package_SO:SOIC-20W_7.5x12.8mm_P1.27mm"
+		(property "Footprint" "Inductor_SMD:L_Cenker_CKCS8040"
 			(at 146.05 72.39 0)
 			(hide yes)
